File: board/board.kicad_pcb (KiCad board)
At the start: 2 copper layers, 54.6 x 61.1 mm, 11 parts, among them J1 RJ45, P8 BeagleBone_Black_Header, P9 BeagleBone_Black_Header, U1 7438

Commit message: Rename boardv2 to board. Replace the Eagle version with the KiCad version
Parts:
- moved J1 5.12 mm to (138.4, 104.1)
Connections:
- R3 pad P$2: Net-(R3-PadP$2) -> /FROM_ALTO
- R4 pad P$1: Net-(R3-PadP$2) -> /FROM_ALTO
Routing:
- net +3V3: track 108.3 -> 58.7 mm
- net /FROM_ALTO: track 28.8 -> 49.1 mm
- net Net-(R3-PadP$2): track 4.19 -> 0.00 mm
- net /TO_ALTO: track 38.7 -> 35.7 mm
- net /COLLISION: track 20.7 -> 17.6 mm
Changed lines of the file:
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@@
 (kicad_pcb (version 4) (host pcbnew 4.0.2-stable)
   (general
-    (links 39)
+    (links 40)
     (no_connects 0)
-    (area 106.380794 56.205 174.619407 120.904001)
+    (area 106.380794 58.205 174.619407 120.904001)
     (thickness 1.6)
     (drawings 14)
-    (tracks 53)
+    (tracks 51)
     (zones 0)
     (modules 11)
-    (nets 90)
+    (nets 89)
   )
   (page USLetter)
   (layers
-    (0 F.Cu signal hide)
-    (31 B.Cu signal)
+    (0 F.Cu signal)
+    (31 B.Cu signal hide)
     (34 B.Paste user hide)
     (35 F.Paste user hide)
@@
   )
   (setup
-    (last_trace_width 0.3048)
+    (last_trace_width 0.1524)
     (user_trace_width 0.3048)
     (trace_clearance 0.1524)
@@
     (pad_to_mask_clearance 0)
     (aux_axis_origin 0 0)
-    (visible_elements 7FFFFFFF)
+    (visible_elements 7FFFEFFF)
     (pcbplotparams
       (layerselection 0x010f0_80000001)
@@
   (net 85 "Net-(P9-Pad32)")
   (net 86 "Net-(P9-Pad34)")
-  (net 87 "Net-(R3-PadP$2)")
-  (net 88 "Net-(U1-Pad8)")
-  (net 89 "Net-(U1-Pad11)")
+  (net 87 "Net-(U1-Pad8)")
+  (net 88 "Net-(U1-Pad11)")
   (net_class Default "To jest domyślna klasa połączeń."
     (clearance 0.1524)
@@
     (add_net "Net-(P9-Pad8)")
     (add_net "Net-(P9-Pad9)")
-    (add_net "Net-(R3-PadP$2)")
     (add_net "Net-(U1-Pad11)")
     (add_net "Net-(U1-Pad8)")
@@
   )
   (module Connect:RJ45_8 (layer F.Cu)
-    (at 133.3119 104.04094)
+    (at 138.43 104.14)
     (tags RJ45)
     (fp_text reference J1 (at 4.7 11.18) (layer F.SilkS)
@@
       (net 72 +3V3) (solder_mask_margin 0.1016))
     (pad P$2 thru_hole circle (at 3.81 0 270) (size 1.8796 1.8796) (drill 0.89916) (layers *.Cu *.Mask)
-      (net 87 "Net-(R3-PadP$2)") (solder_mask_margin 0.1016))
+      (net 78 /FROM_ALTO) (solder_mask_margin 0.1016))
   )
   (module SparkFun:AXIAL-0.3 (layer F.Cu)
@@
     (fp_line (start -2.54 0) (end -2.794 0) (layer F.SilkS) (width 0.2032))
     (pad P$1 thru_hole circle (at -3.81 0 90) (size 1.8796 1.8796) (drill 0.89916) (layers *.Cu *.Mask)
-      (net 87 "Net-(R3-PadP$2)") (solder_mask_margin 0.1016))
+      (net 78 /FROM_ALTO) (solder_mask_margin 0.1016))
     (pad P$2 thru_hole circle (at 3.81 0 90) (size 1.8796 1.8796) (drill 0.89916) (layers *.Cu *.Mask)
       (net 75 GND) (solder_mask_margin 0.1016))
@@
       (net 79 /P8_11))
     (pad 8 thru_hole oval (at 7.62 15.24) (size 1.6 1.6) (drill 0.8) (layers *.Cu *.Mask)
-      (net 88 "Net-(U1-Pad8)"))
+      (net 87 "Net-(U1-Pad8)"))
     (pad 2 thru_hole oval (at 0 2.54) (size 1.6 1.6) (drill 0.8) (layers *.Cu *.Mask)
       (net 79 /P8_11))
@@
       (net 80 /P8_12))
     (pad 11 thru_hole oval (at 7.62 7.62) (size 1.6 1.6) (drill 0.8) (layers *.Cu *.Mask)
-      (net 89 "Net-(U1-Pad11)"))
+      (net 88 "Net-(U1-Pad11)"))
     (pad 5 thru_hole oval (at 0 10.16) (size 1.6 1.6) (drill 0.8) (layers *.Cu *.Mask)
       (net 80 /P8_12))
@@
     (effects (font (size 1.5 1.5) (thickness 0.2032)))
   )
-  (gr_text "Warning:\nNot a standard\nEthernet port\n" (at 126.19482 108.79836 270) (layer F.SilkS)
+  (gr_text "Warning:\nNot a standard\nEthernet port\n" (at 130.81 109.22 270) (layer F.SilkS)
     (effects (font (size 1.5 1.5) (thickness 0.3)))
   )
@@
   (gr_line (start 169.0751 120.8151) (end 169.0751 59.7027) (layer Edge.Cuts) (width 0.00254))
   (gr_line (start 114.4651 59.7027) (end 114.4651 120.8151) (layer Edge.Cuts) (width 0.00254))
+  (segment (start 147.32 96.52) (end 148.59 97.79) (width 0.3048) (layer F.Cu) (net 72))
+  (segment (start 148.59 97.79) (end 155.615 97.79) (width 0.3048) (layer F.Cu) (net 72))
+  (segment (start 147.790001 96.990001) (end 147.32 96.52) (width 0.3048) (layer F.Cu) (net 72))
+  (segment (start 147.32 96.52) (end 144.78 93.98) (width 0.3048) (layer F.Cu) (net 72))
+  (segment (start 134.8577 80.87) (end 134.8577 84.0577) (width 0.3048) (layer F.Cu) (net 72))
+  (segment (start 134.8577 84.0577) (end 144.78 93.98) (width 0.3048) (layer F.Cu) (net 72))
+  (segment (start 118.9101 64.9224) (end 134.8577 80.87) (width 0.3048) (layer F.Cu) (net 72))
   (segment (start 116.3701 64.9224) (end 118.9101 64.9224) (width 0.3048) (layer F.Cu) (net 72))
-  (segment (start 118.9101 64.9224) (end 134.8577 80.87) (width 0.3048) (layer F.Cu) (net 72))
-  (segment (start 151.653339 85.851589) (end 151.653339 93.828339) (width 0.3048) (layer F.Cu) (net 72))
-  (segment (start 134.8577 80.87) (end 146.67175 80.87) (width 0.3048) (layer F.Cu) (net 72))
-  (segment (start 146.67175 80.87) (end 151.653339 85.851589) (width 0.3048) (layer F.Cu) (net 72))
-  (segment (start 151.653339 93.828339) (end 154.815001 96.990001) (width 0.3048) (layer F.Cu) (net 72))
-  (segment (start 154.815001 96.990001) (end 155.615 97.79) (width 0.3048) (layer F.Cu) (net 72))
-  (segment (start 123.36 69.3723) (end 134.989532 81.001832) (width 0.1524) (layer F.Cu) (net 72))
-  (segment (start 134.989532 81.001832) (end 146.690806 81.001832) (width 0.1524) (layer F.Cu) (net 72))
-  (segment (start 146.690806 81.001832) (end 151.729539 86.040565) (width 0.1524) (layer F.Cu) (net 72))
-  (segment (start 151.729539 86.040565) (end 151.729539 93.904539) (width 0.1524) (layer F.Cu) (net 72))
-  (segment (start 151.729539 93.904539) (end 154.815001 96.990001) (width 0.1524) (layer F.Cu) (net 72))
   (segment (start 155.615 97.79) (end 155.615 100.29) (width 0.1524) (layer F.Cu) (net 72))
   (segment (start 155.615 100.29) (end 155.067 100.838) (width 0.1524) (layer F.Cu) (net 72))
@@
   (segment (start 144.272 85.6615) (end 146.94662 82.98688) (width 0.1524) (layer B.Cu) (net 74))
   (segment (start 146.94662 82.98688) (end 146.94662 89.13622) (width 0.1524) (layer B.Cu) (net 74))
-  (segment (start 146.94662 89.13622) (end 134.5819 101.50094) (width 0.1524) (layer B.Cu) (net 74))
+  (segment (start 146.94662 89.13622) (end 139.7 101.6) (width 0.1524) (layer B.Cu) (net 74) (status 20))
   (segment (start 146.94662 82.98688) (end 146.94662 79.22006) (width 0.1524) (layer B.Cu) (net 74))
   (segment (start 146.94662 79.22006) (end 150.25116 79.22006) (width 0.1524) (layer F.Cu) (net 74))
@@
   (segment (start 158.115 97.79) (end 158.115 99.695) (width 0.1524) (layer F.Cu) (net 75))
   (segment (start 158.115 99.695) (end 159.258 100.838) (width 0.1524) (layer F.Cu) (net 75))
-  (segment (start 137.1219 101.50094) (end 149.2758 89.34704) (width 0.1524) (layer B.Cu) (net 76))
+  (segment (start 142.24 101.6) (end 149.2758 89.34704) (width 0.1524) (layer B.Cu) (net 76) (status 10))
   (segment (start 149.2758 89.34704) (end 152.75814 89.34704) (width 0.1524) (layer B.Cu) (net 76))
-  (segment (start 142.2019 101.50094) (end 141.08684 102.616) (width 0.1524) (layer F.Cu) (net 78))
-  (segment (start 141.08684 102.616) (end 131.2037 102.616) (width 0.1524) (layer F.Cu) (net 78))
-  (segment (start 131.2037 102.616) (end 119.773699 91.185999) (width 0.1524) (layer F.Cu) (net 78))
-  (segment (start 119.773699 91.185999) (end 118.9101 90.3224) (width 0.1524) (layer F.Cu) (net 78))
+  (segment (start 118.9101 90.3224) (end 136.0424 90.3224) (width 0.1524) (layer F.Cu) (net 78))
+  (segment (start 136.0424 90.3224) (end 147.32 101.6) (width 0.1524) (layer F.Cu) (net 78))
+  (segment (start 155.067 108.458) (end 154.178 108.458) (width 0.1524) (layer F.Cu) (net 78))
+  (segment (start 155.067 108.458) (end 148.209 101.6) (width 0.1524) (layer F.Cu) (net 78))
+  (segment (start 148.209 101.6) (end 147.32 101.6) (width 0.1524) (layer F.Cu) (net 78))
+  (segment (start 155.067 108.458) (end 155.067 108.077) (width 0.1524) (layer F.Cu) (net 78))
+  (segment (start 159.258 108.458) (end 155.067 108.458) (width 0.1524) (layer F.Cu) (net 78))
   (segment (start 152.75814 76.64704) (end 152.75814 79.18704) (width 0.1524) (layer F.Cu) (net 79))
   (segment (start 164.6301 75.0824) (end 153.37038 75.0824) (width 0.1524) (layer F.Cu) (net 79))
@@
   (segment (start 160.389071 78.158439) (end 158.866741 78.158439) (width 0.1524) (layer F.Cu) (net 80))
   (segment (start 153.558139 83.467041) (end 152.75814 84.26704) (width 0.1524) (layer F.Cu) (net 80))
-  (segment (start 159.258 108.458) (end 155.067 108.458) (width 0.1524) (layer F.Cu) (net 87))
   (zone (net 75) (net_name GND) (layer F.Cu) (hatch edge 0.508)
     (connect_pads (clearance 0.508))
